Commit message: Nuovo bluerov descr

File: urdf/bluerov.urdf.xacro (robot description, xacro)
@@ -1,4 +1,4 @@
 <?xml version="1.0"?>
-<robot name="bluerov" xmlns:xacro="http://www.ros.org/wiki/xacro">
+<robot name="bluerov" family="underwater" xmlns:xacro="http://www.ros.org/wiki/xacro">
   <xacro:arg name="robot_namespace" default="bluerov"/>
   <xacro:arg name="environment" default="real"/>
@@ -29,20 +29,24 @@
     </joint>
   </xacro:macro>
-  <xacro:macro name="ros2_control_thruster_joint" params="joint_name inverted">
-    <joint name="${robot_prefix}${joint_name}">
-      <command_interface name="effort"/>
-      <state_interface name="effort"/>
-      <param name="inverted">${inverted}</param>
-    </joint>
-  </xacro:macro>
+  <xacro:macro name="ros2_control_thruster_joint" params="joint_name inverted channel">
+  <joint name="${robot_prefix}${joint_name}">
+    <command_interface name="effort"/>
+    <state_interface name="effort"/>
+    <param name="lookup_csv">$(arg lookup_csv)</param>
+    <param name="stonefish_topic">$(arg stonefish_topic)</param>
+    <param name="channel">${channel}</param>
+    <param name="inverted">${inverted}</param>
+  </joint>
+</xacro:macro>
 <!-- This macro is defined for future use if we want to add servo motors to the ROV. -->
-<xacro:macro name="ros2_control_servo_joint" params="joint_name inverted center_offset_rad">
-    <joint name="${robot_prefix}${joint_name}">
-      <command_interface name="position"/>
-      <state_interface name="position"/>
-      <param name="inverted">${inverted}</param>
-      <param name="center_offset_rad">${center_offset_rad}</param>
-    </joint>
-  </xacro:macro>
+<xacro:macro name="ros2_control_servo_joint" params="joint_name controller inverted center_offset_rad">
+  <joint name="${robot_prefix}${joint_name}">
+    <command_interface name="position"/>
+    <state_interface name="position"/>
+    <param name="controller">${controller}</param>
+    <param name="inverted">${inverted}</param>
+    <param name="center_offset_rad">${center_offset_rad}</param>
+  </joint>
+</xacro:macro>
 <!-- End of servo joint macro -->
   <link name="${robot_prefix}base_link">
@@ -193,12 +197,12 @@
       <param name="pwm_channels">$(arg pwm_channels)</param>
     </hardware>
-    <xacro:ros2_control_thruster_joint joint_name="Thruster_R_FORWARD_FRONT" inverted="false"/>
-    <xacro:ros2_control_thruster_joint joint_name="Thruster_L_FORWARD_FRONT" inverted="false"/>
-    <xacro:ros2_control_thruster_joint joint_name="Thruster_R_FORWARD_REAR" inverted="true"/>
-    <xacro:ros2_control_thruster_joint joint_name="Thruster_L_FORWARD_REAR" inverted="true"/>
-    <xacro:ros2_control_thruster_joint joint_name="Thruster_R_UP_FRONT" inverted="false"/>
-    <xacro:ros2_control_thruster_joint joint_name="Thruster_L_UP_FRONT" inverted="true"/>
-    <xacro:ros2_control_thruster_joint joint_name="Thruster_R_UP_REAR" inverted="false"/>
-    <xacro:ros2_control_thruster_joint joint_name="Thruster_L_UP_REAR" inverted="false"/>
+    <xacro:ros2_control_thruster_joint joint_name="Thruster_R_FORWARD_FRONT" inverted="false" channel="0"/>
+    <xacro:ros2_control_thruster_joint joint_name="Thruster_L_FORWARD_FRONT" inverted="false" channel="1"/>
+    <xacro:ros2_control_thruster_joint joint_name="Thruster_R_FORWARD_REAR" inverted="true" channel="2"/>
+    <xacro:ros2_control_thruster_joint joint_name="Thruster_L_FORWARD_REAR" inverted="true" channel="3"/>
+    <xacro:ros2_control_thruster_joint joint_name="Thruster_R_UP_FRONT" inverted="false" channel="4"/>
+    <xacro:ros2_control_thruster_joint joint_name="Thruster_L_UP_FRONT" inverted="true" channel="5"/>
+    <xacro:ros2_control_thruster_joint joint_name="Thruster_R_UP_REAR" inverted="false" channel="6"/>
+    <xacro:ros2_control_thruster_joint joint_name="Thruster_L_UP_REAR" inverted="false" channel="7"/>
   </ros2_control>
   <xacro:macro name="ros2_control_sensor_system">
@@ -216,5 +220,7 @@
         <param name="battery_read_rate_hz">1.0</param>
       </hardware>
-      <sensor name="imu_sensor">
+            <sensor name="imu_sensor">
+        <param name="interface">sura_hardware_interface/ImuInterface</param>
+        <param name="stonefish_topic">/${robot_namespace}/stonefish/sensors/imu</param>
         <state_interface name="orientation.x"/>
         <state_interface name="orientation.y"/>
@@ -229,4 +235,6 @@
       </sensor>
       <sensor name="magnetometer_sensor">
+        <param name="interface">sura_hardware_interface/MagnetometerInterface</param>
+        <param name="stonefish_topic">/${robot_namespace}/stonefish/sensors/magnetometer</param>
         <state_interface name="magnetic_field.x"/>
         <state_interface name="magnetic_field.y"/>
@@ -234,7 +242,13 @@
       </sensor>
       <sensor name="pressure_sensor">
+        <param name="interface">sura_hardware_interface/PressureInterface</param>
+        <param name="stonefish_topic">/${robot_namespace}/stonefish/sensors/pressure</param>
+        <param name="pressure_offset_pa">$(arg pressure_offset_pa)</param>
+        <param name="read_rate_hz">200.0</param>
         <state_interface name="fluid_pressure"/>
       </sensor>
       <sensor name="battery_sensor">
+        <param name="interface">sura_hardware_interface/BatteryInterface</param>
+        <param name="read_rate_hz">1.0</param>
         <state_interface name="voltage"/>
         <state_interface name="current"/>
@@ -252,7 +266,7 @@
     </hardware>
     <!-- the order is important: must match the PWM channel order -->
-    <xacro:ros2_control_servo_joint joint_name="newton_gripper_joint" inverted="false" center_offset_rad="0.0"/>
-    <xacro:ros2_control_servo_joint joint_name="servo_zip_joint" inverted="false" center_offset_rad="0.0"/>
-    <xacro:ros2_control_servo_joint joint_name="servo_camera_joint" inverted="false" center_offset_rad="0.0"/>
+    <xacro:ros2_control_servo_joint joint_name="newton_gripper_joint" controller="newton_gripper_controller" inverted="false" center_offset_rad="0.0"/>
+<xacro:ros2_control_servo_joint joint_name="servo_zip_joint" controller="servo_zip_controller" inverted="false" center_offset_rad="0.0"/>
+<xacro:ros2_control_servo_joint joint_name="servo_camera_joint" controller="servo_camera_controller" inverted="false" center_offset_rad="0.0"/>
   </ros2_control>
 </robot>

Commit message: aggiornamento dal bluerov2

File: urdf/bluerov.urdf.xacro (robot description, xacro)
@@ -9,5 +9,5 @@
   <!-- Servo motor parameters for future use -->
   <xacro:arg name="servo_sim_topic" default="/bluerov/controller/servo_setpoints_sim"/>
-  <xacro:arg name="servo_pwm_channels" default="12,14,15"/> <!-- Newton Gripper: 12, Zip = 14,Camera = 15 -->
+  <xacro:arg name="servo_pwm_channels" default="13,14,15"/> <!-- motor Gripper: 13, Zip = 14,Camera = 15 -->
   <!-- End of servo motor parameters -->
   <xacro:property name="robot_namespace" value="$(arg robot_namespace)"/>
@@ -104,4 +104,17 @@
     <origin xyz="0.0 0.0 0.0" rpy="-1.57 3.14 -1.57"/>
   </joint>
+  <!-- camera gripper -->
+  <link name="${robot_prefix}camera_gripper"/>
+  <joint name="${robot_prefix}camera_gripper_joint" type="fixed">
+    <parent link="${robot_prefix}base_link"/>
+    <child link="${robot_prefix}camera_gripper"/>
+    <origin xyz="0.17 -0.005 -0.035" rpy="0.0 0.0 0.0"/>
+  </joint>
+  <link name="${robot_prefix}camera_gripper/optical_frame"/>
+  <joint name="${robot_prefix}camera_gripper_optical_frame_joint" type="fixed">
+    <parent link="${robot_prefix}camera_gripper"/>
+    <child link="${robot_prefix}camera_gripper/optical_frame"/>
+    <origin xyz="0.0 0.0 0.0" rpy="-1.57 3.14 -1.57"/>
+  </joint>
   <!-- camera left -->
   <link name="${robot_prefix}camera_left"/>
@@ -158,12 +171,13 @@
     rpy="1.57 1.57 0.0"/>
   <!-- Newton Gripper -->
-  <link name="${robot_prefix}newton_gripper"/>
-  <joint name="${robot_prefix}newton_gripper_joint" type="prismatic">
-    <parent link="${robot_prefix}base_link"/>
-    <child link="${robot_prefix}newton_gripper"/>
+  <!--<link name="${robot_prefix}newton_gripper"/>-->
+  <!-- Motor Gripper -->
+  <link name="${robot_prefix}motor_gripper"/>
+  <joint name="${robot_prefix}motor_gripper_joint" type="revolute">
+    <parent link="${robot_prefix}base_link"/>
+    <child link="${robot_prefix}motor_gripper"/>
     <origin xyz="0.25 0.0 -0.05" rpy="0.0 0.0 0.0"/>
-    <axis xyz="1 0 0"/>
-    <!-- Limits normalized: da -1.0 a 1.0 -->
-    <limit lower="-1.0" upper="1.0" effort="10.0" velocity="1.0"/>
+    <axis xyz="0 0 1"/>
+    <limit lower="-1.0" upper="1.0" effort="10.0" velocity="10.0"/>
   </joint>
   <!-- Servo Zip -->
@@ -217,10 +231,14 @@
         <param name="sim_gps_topic">/${robot_namespace}/stonefish/sensors/gps</param>
         <param name="pressure_offset_pa">$(arg pressure_offset_pa)</param>
-        <param name="pressure_read_rate_hz">200.0</param>
+        <param name="pressure_read_rate_hz">100.0</param>
         <param name="battery_read_rate_hz">1.0</param>
       </hardware>
-            <sensor name="imu_sensor">
+      <sensor name="imu_sensor">
         <param name="interface">sura_hardware_interface/ImuInterface</param>
+        <param name="broadcaster">imu_broadcaster</param>
+        <param name="read_rate_hz">100.0</param>
+        <param name="frame_id">${robot_namespace}/imu_link</param>
         <param name="stonefish_topic">/${robot_namespace}/stonefish/sensors/imu</param>
+        <param name="msg_type">sensor_msgs/msg/Imu</param>
         <state_interface name="orientation.x"/>
         <state_interface name="orientation.y"/>
@@ -233,17 +251,25 @@
         <state_interface name="linear_acceleration.y"/>
         <state_interface name="linear_acceleration.z"/>
+        <state_interface name="sample_time.sec"/>
+        <state_interface name="sample_time.nanosec"/>
       </sensor>
       <sensor name="magnetometer_sensor">
         <param name="interface">sura_hardware_interface/MagnetometerInterface</param>
+        <param name="broadcaster">magnetometer_broadcaster</param>
+        <param name="read_rate_hz">100.0</param>
+        <param name="frame_id">${robot_namespace}/imu_link</param>
         <param name="stonefish_topic">/${robot_namespace}/stonefish/sensors/magnetometer</param>
+        <param name="msg_type">sensor_msgs/msg/MagneticField</param>
         <state_interface name="magnetic_field.x"/>
         <state_interface name="magnetic_field.y"/>
         <state_interface name="magnetic_field.z"/>
-      </sensor>
+        <state_interface name="sample_time.sec"/>
+        <state_interface name="sample_time.nanosec"/>
+    </sensor>
       <sensor name="pressure_sensor">
         <param name="interface">sura_hardware_interface/PressureInterface</param>
         <param name="stonefish_topic">/${robot_namespace}/stonefish/sensors/pressure</param>
         <param name="pressure_offset_pa">$(arg pressure_offset_pa)</param>
-        <param name="read_rate_hz">200.0</param>
+        <param name="read_rate_hz">100.0</param>
         <state_interface name="fluid_pressure"/>
       </sensor>
@@ -266,7 +292,7 @@
     </hardware>
     <!-- the order is important: must match the PWM channel order -->
-    <xacro:ros2_control_servo_joint joint_name="newton_gripper_joint" controller="newton_gripper_controller" inverted="false" center_offset_rad="0.0"/>
-<xacro:ros2_control_servo_joint joint_name="servo_zip_joint" controller="servo_zip_controller" inverted="false" center_offset_rad="0.0"/>
-<xacro:ros2_control_servo_joint joint_name="servo_camera_joint" controller="servo_camera_controller" inverted="false" center_offset_rad="0.0"/>
+    <xacro:ros2_control_servo_joint joint_name="motor_gripper_joint" controller="motor_gripper_controller" inverted="false" center_offset_rad="0.0"/>
+    <xacro:ros2_control_servo_joint joint_name="servo_zip_joint" controller="servo_zip_controller" inverted="false" center_offset_rad="0.0"/>
+    <xacro:ros2_control_servo_joint joint_name="servo_camera_joint" controller="servo_camera_controller" inverted="false" center_offset_rad="0.0"/>
   </ros2_control>
 </robot>

Commit message: s

File: urdf/bluerov.urdf.xacro (robot description, xacro)
@@ -40,5 +40,5 @@
 </xacro:macro>
 <!-- This macro is defined for future use if we want to add servo motors to the ROV. -->
-<xacro:macro name="ros2_control_servo_joint" params="joint_name controller inverted center_offset_rad">
+<xacro:macro name="ros2_control_servo_joint" params="joint_name controller inverted center_offset_rad pulse_min_us:=1000.0 pulse_max_us:=2000.0">
   <joint name="${robot_prefix}${joint_name}">
     <command_interface name="position"/>
@@ -47,4 +47,6 @@
     <param name="inverted">${inverted}</param>
     <param name="center_offset_rad">${center_offset_rad}</param>
+    <param name="pulse_min_us">${pulse_min_us}</param>
+    <param name="pulse_max_us">${pulse_max_us}</param>
   </joint>
 </xacro:macro>
@@ -292,5 +294,5 @@
     </hardware>
     <!-- the order is important: must match the PWM channel order -->
-    <xacro:ros2_control_servo_joint joint_name="motor_gripper_joint" controller="motor_gripper_controller" inverted="false" center_offset_rad="0.0"/>
+    <xacro:ros2_control_servo_joint joint_name="motor_gripper_joint" controller="motor_gripper_controller" inverted="false" center_offset_rad="0.0" pulse_min_us="500.0" pulse_max_us="2500.0"/>
     <xacro:ros2_control_servo_joint joint_name="servo_zip_joint" controller="servo_zip_controller" inverted="false" center_offset_rad="0.0"/>
     <xacro:ros2_control_servo_joint joint_name="servo_camera_joint" controller="servo_camera_controller" inverted="false" center_offset_rad="0.0"/>
